File: minimouse.kicad_pcb (KiCad board)
At the start: 2 copper layers, 90 x 85 mm, 22 parts, among them J1 Conn_ARM_JTAG_SWD_10, J5 Conn_01x02, M1 N20_encoder, M2 N20_encoder, U1 STM32F030C8Tx, U4 HC-SR04

Commit message: TP3
Parts:
- removed R7: 100, Resistor_SMD:R_0603_1608Metric
- added C10: 1m, Capacitor_SMD:C_0603_1608Metric, F.Cu at (179.7, 102.5)
- added C11: 2.2uF, Capacitor_SMD:C_0603_1608Metric, F.Cu at (234.6, 70.5)
- added C12: 2.2uF, Capacitor_SMD:C_0603_1608Metric, F.Cu at (136.6, 88.8)
- added C13: 2.2uF, Capacitor_SMD:C_0603_1608Metric, F.Cu at (177.2, 76.1)
- added C40: 2.2uF, Capacitor_SMD:C_0603_1608Metric, F.Cu at (155.9, 89.8)
- added C7: C, Capacitor_SMD:C_0603_1608Metric, F.Cu at (122.1, 100.0)
- added C8: 2.2µF, Capacitor_SMD:C_0603_1608Metric, F.Cu at (168.6, 102.5)
- added C9: C, Capacitor_SMD:C_0603_1608Metric, F.Cu at (116.2, 89.8)
- added CS1: 2.2u, Capacitor_SMD:C_0603_1608Metric, F.Cu at (125.4, 84.8)
- added CSTBY1: 10n, Capacitor_SMD:C_0603_1608Metric, F.Cu at (220.8, 58.6)
- added CSTBY2: 10n, Capacitor_SMD:C_0603_1608Metric, F.Cu at (124.8, 97.5)
- added J2: Conn_01x06, Connector_PinHeader_2.54mm:PinHeader_1x06_P2.54mm_Vertical, F.Cu at (172.9, 77.1)
- added J3: Conn_01x04, Connector_PinHeader_2.54mm:PinHeader_1x04_P2.54mm_Vertical, F.Cu at (124.6, 72.1)
- added J4: Conn_01x06, Connector_PinHeader_2.54mm:PinHeader_1x06_P2.54mm_Vertical, F.Cu at (132.2, 89.8)
- added R10: R, Resistor_SMD:R_0603_1608Metric, F.Cu at (111.2, 87.3)
- added R11: R, Resistor_SMD:R_0603_1608Metric, F.Cu at (128.9, 73.5)
- added R12: R, Resistor_SMD:R_0603_1608Metric, F.Cu at (111.2, 92.4)
- added R13: R, Resistor_SMD:R_0603_1608Metric, F.Cu at (234.6, 73.0)
- added R14: 100, Resistor_SMD:R_0603_1608Metric, F.Cu at (136.6, 91.3)
- added R15: 100, Resistor_SMD:R_0603_1608Metric, F.Cu at (136.6, 93.8)
- added R19: 100, Resistor_SMD:R_0603_1608Metric, F.Cu at (177.2, 78.6)
- added R21: 100, Resistor_SMD:R_0603_1608Metric, F.Cu at (177.2, 81.1)
- added ROFF1: 47000, Resistor_SMD:R_0603_1608Metric, F.Cu at (224.8, 58.6)
- added RRCOFF1: 1000, Resistor_SMD:R_0603_1608Metric, F.Cu at (108.5, 97.5)
- added RSNSA1: 0.033, Resistor_SMD:R_0603_1608Metric, F.Cu at (132.2, 79.7)
- added RSNSB1: 0.033, Resistor_SMD:R_0603_1608Metric, F.Cu at (132.2, 82.2)
- added RSTBY1: 18K, Resistor_SMD:R_2512_6332Metric, F.Cu at (118.0, 94.9)
- added U2: STSPIN240, Package_DFN_QFN:VQFN-16-1EP_3x3mm_P0.5mm_EP1.8x1.8mm, F.Cu at (124.5, 91.6)
- added U3: LP5907MFX-3.3, Package_TO_SOT_SMD:SOT-23-5, F.Cu at (174.3, 101.6)
- moved C5 14.0 mm to (112.6, 82.1)
- moved J1 6.89 mm to (157.6, 86.0)
Connections:
- R8 pad 1: /mcu/UART1_TX -> /external_uart/EXT_UART_RX
- U1 pad 19: Net-(U1-PB1) -> /mcu/OUT_B1
- U1 pad 43: /mcu/UART1_RX -> /external_uart/EXT_UART_TX
- U4 pad 2: /mcu/OUT_B9 -> Net-(U4-TRIG)
- U4 pad 3: Net-(U4-ECHO) -> /mcu/TIM8_CH2
- U4 pad 4: +3V3 -> +BATT

Commit message: save
Parts:
- removed C12: 2.2uF, Capacitor_SMD:C_0603_1608Metric
- removed C7: C, Capacitor_SMD:C_0603_1608Metric
- removed CS1: 2.2u, Capacitor_SMD:C_0603_1608Metric
- removed CSTBY1, CSTBY2: 10n, Capacitor_SMD:C_0603_1608Metric
- removed ROFF1: 47000, Resistor_SMD:R_0603_1608Metric
- removed RRCOFF1: 1000, Resistor_SMD:R_0603_1608Metric
- removed RSNSA1, RSNSB1: 0.033, Resistor_SMD:R_0603_1608Metric
- removed RSTBY1: 18K, Resistor_SMD:R_2512_6332Metric
- added C14: 2.2uF, Capacitor_SMD:C_0603_1608Metric, F.Cu at (136.5, 100.0)
- added C15: 2.2uF, Capacitor_SMD:C_0603_1608Metric, F.Cu at (155.1, 74.6)
- added D1: LED, LED_SMD:LED_0603_1608Metric, F.Cu at (178.7, 97.5)
- added R16: 47k, Resistor_SMD:R_0603_1608Metric, F.Cu at (128.9, 84.8)
- added R17: 10k, Resistor_SMD:R_0603_1608Metric, F.Cu at (125.4, 97.5)
- added R20: 100, Resistor_SMD:R_0603_1608Metric, F.Cu at (139.1, 78.8)
- added R22: 100, Resistor_SMD:R_0603_1608Metric, F.Cu at (139.0, 74.6)
- added R23: 100, Resistor_SMD:R_0603_1608Metric, F.Cu at (152.5, 73.8)
- added R7: 330, Resistor_SMD:R_0603_1608Metric, F.Cu at (173.7, 97.5)
- C10: value 1m -> 22nF
- C11: value 2.2uF -> 1nF
- C9: value C -> 1m
- R10: value R -> 100
- R11, R12: value R -> 330m
- R13: value R -> 10K
- R14: value 100 -> 10K
- R15: value 100 -> 1k
- moved R13 104.0 mm to (132.2, 91.6), turned to 180 degrees
- moved C11 89.7 mm to (144.9, 73.4), turned to 90 degrees
- moved C9 54.8 mm to (169.5, 102.5), turned to 180 degrees
- moved C10 49.1 mm to (133.0, 87.3)
- moved C8 19.7 mm to (148.8, 103.1), turned to 90 degrees
- moved R11 19.1 mm to (126.3, 92.4)
- moved J4 14.8 mm to (124.6, 102.5), turned to 90 degrees
- moved R15 10.1 mm to (128.9, 87.3)
- moved R14 7.86 mm to (128.9, 89.7)
- moved J1 6.35 mm to (164.0, 86.0)
- moved R19 4.42 mm to (179.7, 82.2), turned to 180 degrees
- moved R21 4.42 mm to (179.7, 84.8)
- moved U2 2.93 mm to (121.6, 91.6)
- moved R12 2.44 mm to (113.6, 92.4), turned to 180 degrees
Connections:
- C10 pad 1: Net-(U3-OUT) -> Net-(C10-Pad1)
- C11 pad 1: +3.3V -> /mcu/IN_B2
- C40 pad 1: +3.3V -> +BATT
- C9 pad 1: /mcu/OUT_B1 -> +3.3V
- R10 pad 1: /mcu/IN_B2 -> /external_uart/EXT_UART_TX
- R10 pad 2: /mcu/OUT_B1 -> Net-(J3-Pin_3)
- R11 pad 1: /external_uart/EXT_UART_TX -> Net-(U2-SENSEB)
- R11 pad 2: Net-(J3-Pin_3) -> GND
- R12 pad 1: Net-(U2-REF) -> Net-(U2-SENSEA)
- R12 pad 2: +BATT -> GND
- R13 pad 1: /mcu/OUT_B9 -> Net-(U2-REF)
- R13 pad 2: Net-(U4-TRIG) -> +BATT
- R14 pad 1: /mcu/TIM2_CH1 -> GND
- R14 pad 2: Net-(J4-Pin_3) -> Net-(U2-REF)
- R15 pad 1: Net-(J4-Pin_4) -> Net-(U2-TOFF)
- R15 pad 2: /mcu/TIM2_CH2 -> Net-(C10-Pad1)
- U2 pad 13: /mcu/OUT_B1 -> /mcu/IN_B2
- U3 pad 5: Net-(U3-OUT) -> +3.3V
- U4 pad 2: Net-(U4-TRIG) -> /mcu/OUT_B9
- U4 pad 3: /mcu/TIM8_CH2 -> Net-(U4-ECHO)
- U4 pad 4: +BATT -> +3.3V
Routing:
- net +BATT: track 0.00 -> 69.1 mm
- net Net-(U2-TOFF): track 0.00 -> 13.6 mm
- net +3.3V: track 0.00 -> 8.95 mm
- net Net-(J2-Pin_3): track 0.00 -> 5.98 mm
- net Net-(J2-Pin_4): track 0.00 -> 5.97 mm
- net Net-(U2-SENSEA): track 0.00 -> 5.68 mm
- net Net-(D1-A): track 0.00 -> 3.43 mm
- net Net-(C10-Pad1): track 0.00 -> 2.54 mm
- net Net-(U2-SENSEB): track 0.00 -> 2.39 mm
