File: mm_motor_control.kicad_sch (KiCad schematic)
At the start: 0 parts

Commit message: TP3
Parts:
- added C7, C9: C, Capacitor_SMD:C_0603_1608Metric, symbol Device:C
- added CS1: 2.2u, Capacitor_SMD:C_0603_1608Metric, symbol Device:C
- added CSTBY1, CSTBY2: 10n, Capacitor_SMD:C_0603_1608Metric, symbol Device:C
- added R10, R12: R, Resistor_SMD:R_0603_1608Metric, symbol Device:R
- added ROFF1: 47000, Resistor_SMD:R_0603_1608Metric, symbol Device:R
- added RRCOFF1: 1000, Resistor_SMD:R_0603_1608Metric, symbol Device:R
- added RSNSA1, RSNSB1: 0.033, Resistor_SMD:R_0603_1608Metric, symbol Device:R
- added RSTBY1: 18K, Resistor_SMD:R_2512_6332Metric, symbol Device:R
- added U2: STSPIN240, Package_DFN_QFN:VQFN-16-1EP_3x3mm_P0.5mm_EP1.8x1.8mm, symbol Driver_Motor:STSPIN240
Connections:
- net EN: now also C9.1, R10.2, U2.13 (EN/FLT)
- net FAULT: now also R10.1
- net OUT_A1: now also U2.3 (OUTA1)
- net OUT_A2: now also U2.5 (OUTA2)
- net OUT_B1: now also U2.10 (OUTB1)
- net OUT_B2: now also U2.8 (OUTB2)
- net PHASE_A: now also U2.1 (PHA)
- net PHASE_B: now also U2.15 (PHB)
- net PWM_A: now also U2.2 (PWMA)
- net PWM_B: now also U2.16 (PWMB)
- net STBY/RESET: now also CSTBY2.1, RSTBY1.1, U2.14 (STBY/RESET)
- new net: CSTBY1.1, R12.1, U2.11 (REF)
- new net: RSNSB1.1, U2.9 (SENSEB)
- new net: ROFF1.1, RRCOFF1.1, U2.12 (TOFF)
- new net: C7.1, RRCOFF1.2
- new net: RSNSA1.1, U2.4 (SENSEA)
- new net +3.3V: RSTBY1.2
- new net +BATT: CS1.2, R12.2, U2.6 (VS)
- new net GND: C7.2, C9.2, CS1.1, CSTBY1.2, CSTBY2.2, ROFF1.2, RSNSA1.2, RSNSB1.2, U2.17 (EPAD), U2.7 (GND)

Commit message: save
Parts:
- removed CS1: 2.2u, Capacitor_SMD:C_0603_1608Metric, symbol Device:C
- removed CSTBY1, CSTBY2: 10n, Capacitor_SMD:C_0603_1608Metric, symbol Device:C
- removed RSTBY1: 18K, Resistor_SMD:R_2512_6332Metric, symbol Device:R
- added R14: 10K, Resistor_SMD:R_0603_1608Metric, symbol Device:R
- C10: renamed from C7; value C -> 22nF
- C11: renamed from C9; value C -> 1nF
- R11: renamed from RSNSB1; value 0.033 -> 330m
- R12: renamed from RSNSA1; value 0.033 -> 330m
- R13: renamed from R12; value R -> 10K
- R15: renamed from RRCOFF1; value 1000 -> 1k
- R16: renamed from ROFF1; value 47000 -> 47k
- R17: renamed from R10; value R -> 10k
Connections:
- net EN: now also R17.1; no longer C11.1, R17.2, U2.13 (EN/FLT)
- net FAULT: now also C11.1, R17.2, U2.13 (EN/FLT); no longer R17.1
- net GND: now also R14.1
- net at R13.1, U2.11 (REF): now also R14.2
