File: mm_power.kicad_sch (KiCad schematic)
At the start: 1 part, among them J5 Conn_01x02

Commit message: TP3
Parts:
- added C10: 1m, Capacitor_SMD:C_0603_1608Metric, symbol Device:C
- added C8: 2.2µF, Capacitor_SMD:C_0603_1608Metric, symbol Device:C
- added D1: LED, symbol Device:LED
- added R7: 330, symbol Device:R
- added U3: LP5907MFX-3.3, Package_TO_SOT_SMD:SOT-23-5, symbol Regulator_Linear:LP5907MFX-3.3
Connections:
- net +BATT: now also C8.1, U3.1 (IN), U3.3 (EN)
- net GND: now also C10.2, C8.2, D1.1 (K), U3.2 (GND)
- new net: D1.2 (A), R7.2
- new net +3.3V: C10.1, R7.1, U3.5 (OUT)

Commit message: save
Parts:
- D1: footprint (none) -> LED_SMD:LED_0603_1608Metric
- R7: footprint (none) -> Resistor_SMD:R_0603_1608Metric
- renumbered C10 to C9
Other:
- moved on the sheet: C8, C9, J5
